Commit message: Adding lidar and camera link

File: src/robot_description/urdf/myrobot.urdf (robot description, URDF)
Before this commit: robot myrobot, 6 links, 5 joints
Links:
- added link camera_link, mass 0.05; collision box size=0.02 0.06 0.03; visual box size=0.02 0.06 0.03
- added link lidar_link, mass 0.1; collision cylinder length=0.05 radius=0.04; visual cylinder length=0.05 radius=0.04
Joints:
- added joint camera_joint: type fixed, parent base_link, child camera_link, origin xyz=0.16 0 0.02 rpy=0 0 0
- added joint lidar_joint: type fixed, parent base_link, child lidar_link, origin xyz=0 0 0.065 rpy=0 0 0

Commit message: - Adding SLAM functionality to robot - Fixed an issue with the robot's yaw was different on rviz and gazebo. This is due to the robot having 2 axle (one at the front and the other at the back and the DiffDrive plugin does not handle multiple axle well) - Modified gazebo_launch.py to be able to take an arg where you can define the world for gazebo to load - Added a new slam_world.sdf for SLAM testing

File: src/robot_description/urdf/myrobot.urdf (robot description, URDF)
Before this commit: robot myrobot, 8 links, 7 joints
Links:
- removed link left_back_wheel_link
- removed link left_front_wheel_link
- removed link right_back_wheel_link
- removed link right_front_wheel_link
- added link back_caster_link, mass 0.05; collision sphere radius=0.025; visual sphere radius=0.025
- added link front_caster_link, mass 0.05; collision sphere radius=0.025; visual sphere radius=0.025
- added link left_wheel_link, mass 0.2; collision cylinder length=0.04 radius=0.05; visual cylinder length=0.04 radius=0.05
- added link right_wheel_link, mass 0.2; collision cylinder length=0.04 radius=0.05; visual cylinder length=0.04 radius=0.05
Joints:
- removed joint left_back_wheel_joint
- removed joint left_front_wheel_joint
- removed joint right_back_wheel_joint
- removed joint right_front_wheel_joint
- added joint back_caster_joint: type fixed, parent base_link, child back_caster_link, origin xyz=-0.12 0 -0.025 rpy=0 0 0
- added joint front_caster_joint: type fixed, parent base_link, child front_caster_link, origin xyz=0.12 0 -0.025 rpy=0 0 0
- added joint left_wheel_joint: type continuous, parent base_link, child left_wheel_link, origin xyz=0 0.12 0 rpy=0 0 0, axis 0 1 0
- added joint right_wheel_joint: type continuous, parent base_link, child right_wheel_link, origin xyz=0 -0.12 0 rpy=0 0 0, axis 0 1 0
